Commit message: fix error randomizing

File: ros2-mecanum-control/mecanum_description/urdf/mecanum.urdf.xacro (robot description, xacro)
@@ -8,9 +8,9 @@
   <xacro:property name="base_size_z" value="0.005" />
   <xacro:property name="base_mass" value="0.5" />
-  <xacro:macro name="box_inertia" params="m x y z">
+  <!-- <xacro:macro name="box_inertia" params="m x y z">
     <inertia ixx="${m*(y*y+z*z)/12}" ixy="0" ixz="0"
              iyy="${m*(x*x+z*z)/12}" iyz="0"
              izz="${m*(x*x+z*z)/12}"
-    />
+    /> -->
   <!-- include file -->
   <xacro:include filename="$(find mecanum_description)/urdf/base.xacro"/>

Commit message: edit param robot same mecanum

File: ros2-mecanum-control/mecanum_description/urdf/mecanum.urdf.xacro (robot description, xacro)
@@ -4,13 +4,8 @@
   <xacro:arg name="robot_type" default="omni"/>
   <xacro:property name="type" value="$(arg robot_type)" />
-  <xacro:property name="base_size_x" value="0.25" />
-  <xacro:property name="base_size_y" value="0.15" />
-  <xacro:property name="base_size_z" value="0.005" />
+  <xacro:property name="base_size_x" value="1.560" />
+  <xacro:property name="base_size_y" value="0.931" />
+  <xacro:property name="base_size_z" value="0.05" />
   <xacro:property name="base_mass" value="0.5" />
-  <!-- <xacro:macro name="box_inertia" params="m x y z">
-    <inertia ixx="${m*(y*y+z*z)/12}" ixy="0" ixz="0"
-             iyy="${m*(x*x+z*z)/12}" iyz="0"
-             izz="${m*(x*x+z*z)/12}"
-    /> -->
   <!-- include file -->
   <xacro:include filename="$(find mecanum_description)/urdf/base.xacro"/>
@@ -18,11 +13,13 @@
   <xacro:include filename="$(find mecanum_description)/ros2_control/mecanum_ros2_control.xacro"/>
   <!-- parameters wheel -->
+  <xacro:property name="wheel_radius" value="0.203" />
+  <xacro:property name="wheel_lenght" value="0.05" />
   <link name="base_footprint" />
   <!-- parameters base_link -->
-  <xacro:robot_base parent="base_footprint" child="base" xyz="0 0 0.075" rpy="0 0 0" />
-  <xacro:wheel parent="base" child="fl" xyz="0.10 0.10 -0.04" rpy="1.57 0 0" robot_type="$(arg robot_type)" />
-  <xacro:wheel parent="base" child="fr" xyz="0.10 -0.10 -0.04" rpy="1.57 0 0" robot_type="$(arg robot_type)" />
-  <xacro:wheel parent="base" child="rl" xyz="-0.10 0.10 -0.04" rpy="1.57 0 0" robot_type="$(arg robot_type)" />
-  <xacro:wheel parent="base" child="rr" xyz="-0.10 -0.10 -0.04" rpy="1.57 0 0" robot_type="$(arg robot_type)" />
+  <xacro:robot_base parent="base_footprint" child="base" xyz="0 0 ${wheel_radius}" rpy="0 0 0" />
+  <xacro:wheel parent="base" child="fl" xyz="${base_size_x/2} ${base_size_y/2} 0" rpy="1.57 0 0" robot_type="$(arg robot_type)" />
+  <xacro:wheel parent="base" child="fr" xyz="${base_size_x/2} ${-base_size_y/2} 0" rpy="1.57 0 0" robot_type="$(arg robot_type)" />
+  <xacro:wheel parent="base" child="rl" xyz="${-base_size_x/2} ${base_size_y/2} 0" rpy="1.57 0 0" robot_type="$(arg robot_type)" />
+  <xacro:wheel parent="base" child="rr" xyz="${-base_size_x/2} ${-base_size_y/2} 0" rpy="1.57 0 0" robot_type="$(arg robot_type)" />
   <xacro:mecanum_ros2_control name="mecanum_robot" use_mock_hardware="true"/>
 </robot>

File: ros2-mecanum-control/mecanum_description/urdf/wheel.xacro (robot description, xacro)
@@ -5,5 +5,5 @@
       <visual>
         <geometry>
-          <cylinder radius="0.0375" length="0.04"/>
+          <cylinder radius="${wheel_radius}" length="${wheel_lenght}"/>
         </geometry>
         <material name="blue">
@@ -13,5 +13,5 @@
       <collision>
         <geometry>
-          <cylinder radius="0.0375" length="0.04"/>
+          <cylinder radius="${wheel_radius}" length="${wheel_lenght}"/>
         </geometry>
       </collision>
