Commit message: edit Readme

File: ros2-mecanum-control/mecanum_description/ros2_control/mecanum_ros2_control.xacro (robot description, xacro)
@@ -5,5 +5,5 @@
       <xacro:unless value="${use_mock_hardware}">
         <hardware>
-          <plugin>mecanumbot_hardware/MecanumbotHardware</plugin>
+          <plugin>mecanum_hardware/MecanumHardware</plugin>
           <!-- <param name="serial_port">/dev/ttyACM0</param> -->
         </hardware>
@@ -11,6 +11,5 @@
       <xacro:if value="${use_mock_hardware}">
         <hardware>
-          <plugin>mecanumbot_hardware/MecanumbotHardware</plugin>
-          <!-- <param name="serial_port">/dev/ttyACM0</param> -->
+          <plugin>mecanum_hardware/MecanumHardware</plugin>
         </hardware>
       </xacro:if>

File: ros2-mecanum-control/mecanum_description/urdf/mecanum.urdf.xacro (robot description, xacro)
@@ -4,5 +4,5 @@
   <xacro:arg name="robot_type" default="omni"/>
   <xacro:property name="type" value="$(arg robot_type)" />
-  <xacro:property name="base_size_x" value="05.25" />
+  <xacro:property name="base_size_x" value="0.25" />
   <xacro:property name="base_size_y" value="0.15" />
   <xacro:property name="base_size_z" value="0.005" />
@@ -16,5 +16,5 @@
   <xacro:include filename="$(find mecanum_description)/urdf/base.xacro"/>
   <xacro:include filename="$(find mecanum_description)/urdf/wheel.xacro"/>
-  <!-- <xacro:include filename="$(find mecanum_description)/ros2_control/mecanum_ros2_control.xacro"/> -->
+  <xacro:include filename="$(find mecanum_description)/ros2_control/mecanum_ros2_control.xacro"/>
   <!-- parameters wheel -->
   <link name="base_footprint" />
@@ -25,4 +25,4 @@
   <xacro:wheel parent="base" child="rl" xyz="-0.10 0.10 -0.04" rpy="1.57 0 0" robot_type="$(arg robot_type)" />
   <xacro:wheel parent="base" child="rr" xyz="-0.10 -0.10 -0.04" rpy="1.57 0 0" robot_type="$(arg robot_type)" />
-  <!-- <xacro:mecanum_ros2_control name="mecanum_robot" use_mock_hardware="true"/> -->
+  <xacro:mecanum_ros2_control name="mecanum_robot" use_mock_hardware="true"/>
 </robot>

File: ros2-mecanum-control/mecanum_description/urdf/wheel.xacro (robot description, xacro)
@@ -22,5 +22,5 @@
     </link>
     <xacro:if value="${robot_type == 'omni'}">
-      <joint name="${child}_joint" type="fixed">
+      <joint name="${child}_joint" type="continuous">
         <axis xyz="0.0 0.0 1"/>
         <origin xyz="${xyz}" rpy="${rpy}" />

Commit message: sửa lại packages mecanum controller

File: ros2-mecanum-control/mecanum_description/ros2_control/mecanum_ros2_control.xacro (robot description, xacro)
@@ -12,4 +12,6 @@
         <hardware>
           <plugin>mecanum_hardware/MecanumHardware</plugin>
+          <param name="example_param_hw_start_duration_sec">0</param>
+          <param name="example_param_hw_stop_duration_sec">3.0</param>
         </hardware>
       </xacro:if>

File: ros2-mecanum-control/mecanum_description/urdf/mecanum.urdf.xacro (robot description, xacro)
@@ -4,7 +4,9 @@
   <xacro:arg name="robot_type" default="omni"/>
   <xacro:property name="type" value="$(arg robot_type)" />
-  <xacro:property name="base_size_x" value="1.560" />
-  <xacro:property name="base_size_y" value="0.931" />
-  <xacro:property name="base_size_z" value="0.05" />
+  <!-- <xacro:property name="base_size_x" value="1.560" />
+  <xacro:property name="base_size_y" value="0.931" /> -->
+  <xacro:property name="base_size_x" value="0.25" />
+  <xacro:property name="base_size_y" value="0.15" />
+  <xacro:property name="base_size_z" value="0.005" />
   <xacro:property name="base_mass" value="0.5" />
   <!-- include file -->
@@ -13,13 +15,15 @@
   <xacro:include filename="$(find mecanum_description)/ros2_control/mecanum_ros2_control.xacro"/>
   <!-- parameters wheel -->
-  <xacro:property name="wheel_radius" value="0.203" />
-  <xacro:property name="wheel_lenght" value="0.05" />
+  <xacro:property name="wheel_radius" value="0.0375" />
+  <xacro:property name="wheel_lenght" value="0.04" />
+  <!-- <xacro:property name="wheel_radius" value="0.203" />
+  <xacro:property name="wheel_lenght" value="0.05" /> -->
   <link name="base_footprint" />
   <!-- parameters base_link -->
-  <xacro:robot_base parent="base_footprint" child="base" xyz="0 0 ${wheel_radius}" rpy="0 0 0" />
-  <xacro:wheel parent="base" child="fl" xyz="${base_size_x/2} ${base_size_y/2} 0" rpy="1.57 0 0" robot_type="$(arg robot_type)" />
-  <xacro:wheel parent="base" child="fr" xyz="${base_size_x/2} ${-base_size_y/2} 0" rpy="1.57 0 0" robot_type="$(arg robot_type)" />
-  <xacro:wheel parent="base" child="rl" xyz="${-base_size_x/2} ${base_size_y/2} 0" rpy="1.57 0 0" robot_type="$(arg robot_type)" />
-  <xacro:wheel parent="base" child="rr" xyz="${-base_size_x/2} ${-base_size_y/2} 0" rpy="1.57 0 0" robot_type="$(arg robot_type)" />
+  <xacro:robot_base parent="base_footprint" child="base" xyz="0 0 ${wheel_radius*2}" rpy="0 0 0" />
+  <xacro:wheel parent="base" child="fl" xyz="${base_size_x/2} ${base_size_y/2} ${-wheel_radius}" rpy="1.57 0 0" robot_type="$(arg robot_type)" />
+  <xacro:wheel parent="base" child="fr" xyz="${base_size_x/2} ${-base_size_y/2} ${-wheel_radius}" rpy="1.57 0 0" robot_type="$(arg robot_type)" />
+  <xacro:wheel parent="base" child="rl" xyz="${-base_size_x/2} ${base_size_y/2} ${-wheel_radius}" rpy="1.57 0 0" robot_type="$(arg robot_type)" />
+  <xacro:wheel parent="base" child="rr" xyz="${-base_size_x/2} ${-base_size_y/2} ${-wheel_radius}" rpy="1.57 0 0" robot_type="$(arg robot_type)" />
   <xacro:mecanum_ros2_control name="mecanum_robot" use_mock_hardware="true"/>
 </robot>
