Commit message: xoa file description tham khao từ nguồn khác và giảm cấp thư mục

File: mecanum_description/urdf/lidar.xacro (robot description, xacro)
@@ -1,28 +1,28 @@
 <?xml version="1.0"?>
 <robot xmlns:xacro="http://wiki.ros.org/xacro">
-  <xacro:macro name="robot_base" params="parent child xyz rpy">
-    <link name="${child}">
+  <xacro:macro name="lidar" params="parent child xyz rpy">
+    <link name="${child}_link">
       <visual>
         <geometry>
-          <box size="0.25 0.15 0.005" />
+          <box size="0.10 0.075 0.060" />
         </geometry>
-        <material name="green">
-          <color rgba="0.0 1 0.0 1" />
+        <material name="blue">
+          <color rgba="0.0 0.0 1 1" />
         </material>
       </visual>
       <collision>
         <geometry>
-          <box size="0.25 0.15 0.005" />
+          <box size="0.10 0.075 0.060" />
         </geometry>
       </collision>
       <inertial>
-        <mass value="0.5" />
+        <mass value="0.01" />
         <inertia ixx="0.015" ixy="0" ixz="0" iyy="0.0375" iyz="0.0" izz="0.0275" />
       </inertial>
     </link>
-    <joint name="${parent}_to_${child}_joint" type="fixed">
+    <joint name="${child}_joint" type="fixed">
       <origin xyz="${xyz}" rpy="${rpy}" />
-      <parent link="${parent}" />
-      <child link="${child}" />
+      <parent link="${parent}_link" />
+      <child link="${child}_link" />
     </joint>
   </xacro:macro>

File: mecanum_description/urdf/mecanum.urdf.xacro (robot description, xacro)
@@ -13,4 +13,5 @@
   <xacro:include filename="$(find mecanum_description)/urdf/base.xacro"/>
   <xacro:include filename="$(find mecanum_description)/urdf/wheel.xacro"/>
+  <xacro:include filename="$(find mecanum_description)/urdf/lidar.xacro"/>
   <xacro:include filename="$(find mecanum_description)/ros2_control/mecanum_ros2_control.xacro"/>
   <!-- parameters wheel -->
@@ -26,4 +27,5 @@
   <xacro:wheel parent="base" child="rl" xyz="${-base_size_x/2} ${base_size_y/2} ${-wheel_radius}" rpy="1.57 0 0" robot_type="$(arg robot_type)" />
   <xacro:wheel parent="base" child="rr" xyz="${-base_size_x/2} ${-base_size_y/2} ${-wheel_radius}" rpy="1.57 0 0" robot_type="$(arg robot_type)" />
+  <xacro:lidar parent="base" child="lidar" xyz="0.04 0.0 0.035" rpy="0 0 0" />
   <xacro:mecanum_ros2_control name="mecanum_robot" use_mock_hardware="true"/>
 </robot>
